File: hardware/Pasta-Pounder-I/Pasta-Pounder-I.kicad_sch (KiCad schematic)
At the start: 57 parts, among them CN1 XT30UPB-M, J1 USB_C_Receptacle, J10 Motor_2-, J11 ESC_VCC, J12 ESC_GND, J4 ESC_Port, J5 JST-SH, J7 Motor_1+, J8 Motor_1-, J9 Motor_2+, Q1 AO3401A, SW1 RESET-SW, SW2 BOOT-SW, SW3 5.8 ZSPT, U1 DRV8874PWPR, U2 DRV8874PWPR, U3 ESP32-S3-MINI-1U, U4 USBLC6-2P6, U7 SY8113BADC

Commit message: Miscelaneous PCB changes
Other:
- company: Carbonara Individuals -> Carbonara Systems
Changed lines of the file:
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@@
 		(title "Pasta Pounder I")
 		(rev "v1.0")
-		(company "Carbonara Individuals")
+		(company "Carbonara Systems")
 		(comment 1 "Developed By: Daniel Principe & Saurya Shrestha")
 	)
